File: electronics/Five_Octave_Keys/Five_Octave_Keys.kicad_pcb (KiCad board)
At the start: 2 copper layers, 0 parts

Commit message: Layout Keys board
Parts:
- added D1: 1N4148WS, Project_Library:D_SOD-323F, F.Cu at (301.7, 38.1)
- added D10: 1N4148WS, Project_Library:D_SOD-323F, F.Cu at (130.2, 38.1)
- added D11: 1N4148WS, Project_Library:D_SOD-323F, F.Cu at (111.2, 38.1)
- added D12: 1N4148WS, Project_Library:D_SOD-323F, F.Cu at (92.1, 38.1)
- added D13: 1N4148WS, Project_Library:D_SOD-323F, F.Cu at (73.1, 38.1)
- added D14: 1N4148WS, Project_Library:D_SOD-323F, F.Cu at (54.0, 38.1)
- added D15: 1N4148WS, Project_Library:D_SOD-323F, F.Cu at (35.0, 38.1)
- added D16: 1N4148WS, Project_Library:D_SOD-323F, F.Cu at (296.9, 57.1)
- added D17: 1N4148WS, Project_Library:D_SOD-323F, F.Cu at (273.1, 57.1)
- added D18: 1N4148WS, Project_Library:D_SOD-323F, F.Cu at (254.0, 57.1)
- added D19: 1N4148WS, Project_Library:D_SOD-323F, F.Cu at (235.0, 57.1)
- added D2: 1N4148WS, Project_Library:D_SOD-323F, F.Cu at (282.6, 38.1)
- added D20: 1N4148WS, Project_Library:D_SOD-323F, F.Cu at (215.9, 57.1)
- added D21: 1N4148WS, Project_Library:D_SOD-323F, F.Cu at (196.9, 57.1)
- added D22: 1N4148WS, Project_Library:D_SOD-323F, F.Cu at (177.8, 57.1)
- added D23: 1N4148WS, Project_Library:D_SOD-323F, F.Cu at (158.8, 57.1)
- added D24: 1N4148WS, Project_Library:D_SOD-323F, F.Cu at (139.7, 57.1)
- added D25: 1N4148WS, Project_Library:D_SOD-323F, F.Cu at (120.7, 57.1)
- added D26: 1N4148WS, Project_Library:D_SOD-323F, F.Cu at (101.6, 57.1)
- added D27: 1N4148WS, Project_Library:D_SOD-323F, F.Cu at (82.6, 57.1)
- added D28: 1N4148WS, Project_Library:D_SOD-323F, F.Cu at (63.5, 57.1)
- added D29: 1N4148WS, Project_Library:D_SOD-323F, F.Cu at (39.7, 57.1)
- added D3: 1N4148WS, Project_Library:D_SOD-323F, F.Cu at (263.6, 38.1)
- added D30: 1N4148WS, Project_Library:D_SOD-323F, F.Cu at (294.5, 76.2)
- added D31: 1N4148WS, Project_Library:D_SOD-323F, F.Cu at (268.3, 76.2)
- added D32: 1N4148WS, Project_Library:D_SOD-323F, F.Cu at (249.3, 76.2)
- added D33: 1N4148WS, Project_Library:D_SOD-323F, F.Cu at (230.2, 76.2)
- added D34: 1N4148WS, Project_Library:D_SOD-323F, F.Cu at (211.2, 76.2)
- added D35: 1N4148WS, Project_Library:D_SOD-323F, F.Cu at (192.1, 76.2)
- added D36: 1N4148WS, Project_Library:D_SOD-323F, F.Cu at (173.1, 76.2)
- added D37: 1N4148WS, Project_Library:D_SOD-323F, F.Cu at (154.0, 76.2)
- added D38: 1N4148WS, Project_Library:D_SOD-323F, F.Cu at (135.0, 76.2)
- added D39: 1N4148WS, Project_Library:D_SOD-323F, F.Cu at (115.9, 76.2)
- added D4: 1N4148WS, Project_Library:D_SOD-323F, F.Cu at (244.5, 38.1)
- added D40: 1N4148WS, Project_Library:D_SOD-323F, F.Cu at (96.9, 76.2)
- added D41: 1N4148WS, Project_Library:D_SOD-323F, F.Cu at (77.8, 76.2)
- added D42: 1N4148WS, Project_Library:D_SOD-323F, F.Cu at (46.9, 76.2)
- added D43: 1N4148WS, Project_Library:D_SOD-323F, F.Cu at (289.8, 95.2)
- added D44: 1N4148WS, Project_Library:D_SOD-323F, F.Cu at (258.8, 95.2)
- added D45: 1N4148WS, Project_Library:D_SOD-323F, F.Cu at (239.8, 95.2)
- added D46: 1N4148WS, Project_Library:D_SOD-323F, F.Cu at (220.7, 95.2)
- added D47: 1N4148WS, Project_Library:D_SOD-323F, F.Cu at (201.7, 95.2)
- added D48: 1N4148WS, Project_Library:D_SOD-323F, F.Cu at (182.6, 95.2)
- added D49: 1N4148WS, Project_Library:D_SOD-323F, F.Cu at (163.6, 95.2)
- added D5: 1N4148WS, Project_Library:D_SOD-323F, F.Cu at (225.5, 38.1)
- added D50: 1N4148WS, Project_Library:D_SOD-323F, F.Cu at (144.5, 95.2)
- added D51: 1N4148WS, Project_Library:D_SOD-323F, F.Cu at (125.5, 95.2)
- added D52: 1N4148WS, Project_Library:D_SOD-323F, F.Cu at (106.4, 95.2)
- added D53: 1N4148WS, Project_Library:D_SOD-323F, F.Cu at (87.4, 95.2)
- added D54: 1N4148WS, Project_Library:D_SOD-323F, F.Cu at (68.3, 95.2)
- added D55: 1N4148WS, Project_Library:D_SOD-323F, F.Cu at (42.1, 95.2)
- added D56: 1N4148WS, Project_Library:D_SOD-323F, F.Cu at (299.3, 114.3)
- added D57: 1N4148WS, Project_Library:D_SOD-323F, F.Cu at (275.5, 114.3)
- added D58: 1N4148WS, Project_Library:D_SOD-323F, F.Cu at (251.7, 114.3)
- added D59: 1N4148WS, Project_Library:D_SOD-323F, F.Cu at (180.2, 114.3)
- added D6: 1N4148WS, Project_Library:D_SOD-323F, F.Cu at (206.4, 38.1)
- added D60: 1N4148WS, Project_Library:D_SOD-323F, F.Cu at (111.2, 114.3)
- added D61: 1N4148WS, Project_Library:D_SOD-323F, F.Cu at (92.1, 114.3)
- added D7: 1N4148WS, Project_Library:D_SOD-323F, F.Cu at (187.4, 38.1)
- added D8: 1N4148WS, Project_Library:D_SOD-323F, F.Cu at (168.3, 38.1)
- added D9: 1N4148WS, Project_Library:D_SOD-323F, F.Cu at (149.3, 38.1)
- added J1: FFC Connector, Project_Library:JUSHUO_AFC01-S16FCC-00, F.Cu at (204.8, 114.3)
- added REF**: Stabilizer_6_25u, Project_Library:Stabilizer_6_25u, F.Cu at (183.4, 114.3)
- added REF**: Stabilizer_2u, Project_Library:Stabilizer_2u, B.Cu at (292.9, 95.2)
- added REF**: Stabilizer_2u, Project_Library:Stabilizer_2u, B.Cu at (50.0, 76.2)
- added SW1: Key Esc, Project_Library:Hot_Swap_Socket_CPG151101S11, F.Cu at (304.8, 38.1)
- added SW10: Key 9, Project_Library:Hot_Swap_Socket_CPG151101S11, F.Cu at (133.3, 38.1)
- added SW11: Key 0, Project_Library:Hot_Swap_Socket_CPG151101S11, F.Cu at (114.3, 38.1)
- added SW12: Key -, Project_Library:Hot_Swap_Socket_CPG151101S11, F.Cu at (95.2, 38.1)
- added SW13: Key =, Project_Library:Hot_Swap_Socket_CPG151101S11, F.Cu at (76.2, 38.1)
- added SW14: Key \, Project_Library:Hot_Swap_Socket_CPG151101S11, F.Cu at (57.1, 38.1)
- added SW15: Key `, Project_Library:Hot_Swap_Socket_CPG151101S11, F.Cu at (38.1, 38.1)
- added SW16: Key Tab, Project_Library:Hot_Swap_Socket_CPG151101S11, F.Cu at (300.0, 57.1)
- added SW17: Key Q, Project_Library:Hot_Swap_Socket_CPG151101S11, F.Cu at (276.2, 57.1)
- added SW18: Key W, Project_Library:Hot_Swap_Socket_CPG151101S11, F.Cu at (257.2, 57.1)
- added SW19: Key E, Project_Library:Hot_Swap_Socket_CPG151101S11, F.Cu at (238.1, 57.1)
- added SW2: Key 1, Project_Library:Hot_Swap_Socket_CPG151101S11, F.Cu at (285.8, 38.1)
- added SW20: Key R, Project_Library:Hot_Swap_Socket_CPG151101S11, F.Cu at (219.1, 57.1)
- added SW21: Key T, Project_Library:Hot_Swap_Socket_CPG151101S11, F.Cu at (200.0, 57.1)
- added SW22: Key Y, Project_Library:Hot_Swap_Socket_CPG151101S11, F.Cu at (181.0, 57.1)
- added SW23: Key U, Project_Library:Hot_Swap_Socket_CPG151101S11, F.Cu at (161.9, 57.1)
- added SW24: Key I, Project_Library:Hot_Swap_Socket_CPG151101S11, F.Cu at (142.9, 57.1)
- added SW25: Key O, Project_Library:Hot_Swap_Socket_CPG151101S11, F.Cu at (123.8, 57.1)
- added SW26: Key P, Project_Library:Hot_Swap_Socket_CPG151101S11, F.Cu at (104.8, 57.1)
- added SW27: Key [, Project_Library:Hot_Swap_Socket_CPG151101S11, F.Cu at (85.7, 57.1)
- added SW28: Key ], Project_Library:Hot_Swap_Socket_CPG151101S11, F.Cu at (66.7, 57.1)
- added SW29: Key BS, Project_Library:Hot_Swap_Socket_CPG151101S11, F.Cu at (42.9, 57.1)
- added SW3: Key 2, Project_Library:Hot_Swap_Socket_CPG151101S11, F.Cu at (266.7, 38.1)
- added SW30: Key Caps, Project_Library:Hot_Swap_Socket_CPG151101S11, F.Cu at (297.7, 76.2)
- added SW31: Key A, Project_Library:Hot_Swap_Socket_CPG151101S11, F.Cu at (271.5, 76.2)
- added SW32: Key S, Project_Library:Hot_Swap_Socket_CPG151101S11, F.Cu at (252.4, 76.2)
- added SW33: Key D, Project_Library:Hot_Swap_Socket_CPG151101S11, F.Cu at (233.4, 76.2)
- added SW34: Key F, Project_Library:Hot_Swap_Socket_CPG151101S11, F.Cu at (214.3, 76.2)
- added SW35: Key G, Project_Library:Hot_Swap_Socket_CPG151101S11, F.Cu at (195.3, 76.2)
- added SW36: Key H, Project_Library:Hot_Swap_Socket_CPG151101S11, F.Cu at (176.2, 76.2)
- added SW37: Key J, Project_Library:Hot_Swap_Socket_CPG151101S11, F.Cu at (157.2, 76.2)
- added SW38: Key K, Project_Library:Hot_Swap_Socket_CPG151101S11, F.Cu at (138.1, 76.2)
- added SW39: Key L, Project_Library:Hot_Swap_Socket_CPG151101S11, F.Cu at (119.1, 76.2)
- added SW4: Key 3, Project_Library:Hot_Swap_Socket_CPG151101S11, F.Cu at (247.7, 38.1)
- added SW40: Key ;, Project_Library:Hot_Swap_Socket_CPG151101S11, F.Cu at (100.0, 76.2)
- added SW41: Key ', Project_Library:Hot_Swap_Socket_CPG151101S11, F.Cu at (81.0, 76.2)
- added SW42: Key Return, Project_Library:Hot_Swap_Socket_CPG151101S11, F.Cu at (50.0, 76.2)
- added SW43: Key Shift, Project_Library:Hot_Swap_Socket_CPG151101S11, F.Cu at (292.9, 95.2)
- added SW44: Key Z, Project_Library:Hot_Swap_Socket_CPG151101S11, F.Cu at (261.9, 95.2)
- added SW45: Key X, Project_Library:Hot_Swap_Socket_CPG151101S11, F.Cu at (242.9, 95.2)
- added SW46: Key C, Project_Library:Hot_Swap_Socket_CPG151101S11, F.Cu at (223.8, 95.2)
- added SW47: Key V, Project_Library:Hot_Swap_Socket_CPG151101S11, F.Cu at (204.8, 95.2)
- added SW48: Key B, Project_Library:Hot_Swap_Socket_CPG151101S11, F.Cu at (185.7, 95.2)
- added SW49: Key N, Project_Library:Hot_Swap_Socket_CPG151101S11, F.Cu at (166.7, 95.2)
- added SW5: Key 4, Project_Library:Hot_Swap_Socket_CPG151101S11, F.Cu at (228.6, 38.1)
- added SW50: Key M, Project_Library:Hot_Swap_Socket_CPG151101S11, F.Cu at (147.6, 95.2)
- added SW51: Key ,, Project_Library:Hot_Swap_Socket_CPG151101S11, F.Cu at (128.6, 95.2)
- added SW52: Key ., Project_Library:Hot_Swap_Socket_CPG151101S11, F.Cu at (109.5, 95.2)
- added SW53: Key /, Project_Library:Hot_Swap_Socket_CPG151101S11, F.Cu at (90.5, 95.2)
- added SW54: Key Shift, Project_Library:Hot_Swap_Socket_CPG151101S11, F.Cu at (71.4, 95.2)
- added SW55: Key Fn, Project_Library:Hot_Swap_Socket_CPG151101S11, F.Cu at (45.2, 95.2)
- added SW56: Key Ctrl, Project_Library:Hot_Swap_Socket_CPG151101S11, F.Cu at (302.4, 114.3)
- added SW57: Key Opt, Project_Library:Hot_Swap_Socket_CPG151101S11, F.Cu at (278.6, 114.3)
- added SW58: Key Cmd, Project_Library:Hot_Swap_Socket_CPG151101S11, F.Cu at (254.8, 114.3)
- added SW59: Key Space, Project_Library:Hot_Swap_Socket_CPG151101S11, F.Cu at (183.4, 114.3)
- added SW6: Key 5, Project_Library:Hot_Swap_Socket_CPG151101S11, F.Cu at (209.6, 38.1)
- added SW60: Key Cmd, Project_Library:Hot_Swap_Socket_CPG151101S11, F.Cu at (114.3, 114.3)
- added SW61: Key MO(1), Project_Library:Hot_Swap_Socket_CPG151101S11, F.Cu at (95.2, 114.3)
- added SW7: Key 6, Project_Library:Hot_Swap_Socket_CPG151101S11, F.Cu at (190.5, 38.1)
- added SW8: Key 7, Project_Library:Hot_Swap_Socket_CPG151101S11, F.Cu at (171.4, 38.1)
- added SW9: Key 8, Project_Library:Hot_Swap_Socket_CPG151101S11, F.Cu at (152.4, 38.1)
Other:
- board outline added: 285.8 x 95.2 mm
