File: electronics/Five_Octave_Keys/Five_Octave_Keys.kicad_pcb (KiCad board)
At the start: 2 copper layers, 285.8 x 95.2 mm, 126 parts, among them J1 FFC Connector, SW1 Key Esc, SW10 Key 9, SW11 Key 0, SW12 Key -, SW13 Key =, SW14 Key \, SW15 Key `, SW16 locked, SW17 Key Q, SW18 locked, SW19 Key E, SW2 Key 1, SW20 Key R, SW21 Key T, SW22 Key Y, SW23 Key U, SW24 Key I, SW25 Key O, SW26 Key P, SW27 Key [, SW28 Key ], SW29 Key BS, SW3 Key 2, SW30 Key Caps, SW31 Key A, SW32 Key S, SW33 Key D, SW34 Key F, SW35 Key G, SW36 Key H, SW37 Key J, SW38 Key K, SW39 Key L, SW4 Key 3, SW40 Key ;, SW41 Key ', SW42 Key Return, SW43 Key Shift, SW44 Key Z, SW45 Key X, SW46 Key C, SW47 Key V, SW48 Key B, SW49 Key N, SW5 Key 4, SW50 Key M, SW51 Key ,, SW52 Key ., SW53 Key /, SW54 Key Shift, SW55 Key Fn, SW56 Key Ctrl, SW57 Key Opt, SW58 Key Cmd, SW59 Key Space, SW6 Key 5, SW60 Key Cmd, SW61 Key MO(1), SW7 Key 6, SW8 Key 7, SW9 Key 8

Commit message: Update
- Assign JLCPCB part number to SW1-61
- GH60 compatible
Parts:
- REF** (x2): moved to F.Cu
- turned REF** to 180 degrees (x2)
Routing:
- net ROW7: track 151.7 -> 176.8 mm, vias 2 -> 4
- added copper zone on B.Cu, net (none)
- added copper zone on F.Cu, net (none)
Other:
- outline, holes or cut-outs redrawn

Commit message: Decorate PCB with silkscreen
Other:
- board text added: "locked"
Changed lines of the file:
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@@
     (title "Five Octave - Keys")
     (date "2023-08-11")
-    (rev "0.4.1-wip.1")
+    (rev "0.4.1-wip.2")
     (comment 1 "https://github.com/takayoshiotake/five-octave-61-key-keyboard")
   )
@@
     (property "ki_keywords" "connector")
     (attr smd)
-    (fp_text reference "J1" (at 0 -2.585 180 unlocked) (layer "F.SilkS")
+    (fp_text reference "J1" (at 0 -2.585 180 unlocked) (layer "F.SilkS") hide
         (effects (font (size 1 1) (thickness 0.15)))
     )
@@
     )
   )
+  (gr_poly
+    (pts
+      (xy 201.91625 106.325)
+      (xy 201.91625 107.325)
+      (xy 199.91625 107.325)
+      (xy 199.91625 108.325)
+      (xy 201.91625 108.325)
+      (xy 201.91625 109.325)
+      (xy 199.91625 109.325)
+      (xy 199.91625 110.325)
+      (xy 201.91625 110.325)
+      (xy 201.91625 109.325)
+      (xy 202.91625 109.325)
+      (xy 202.91625 110.325)
+      (xy 204.91625 110.325)
+      (xy 204.91625 109.325)
+      (xy 202.91625 109.325)
+      (xy 202.91625 108.325)
+      (xy 204.91625 108.325)
+      (xy 204.91625 107.325)
+      (xy 202.91625 107.325)
+      (xy 202.91625 106.325)
+    )
+    (stroke (width 0) (type solid)) (fill solid) (layer "F.Cu"))
+  (gr_rect (start 199.91625 105.325) (end 200.91625 106.325)
+    (stroke (width 0) (type solid)) (fill solid) (layer "F.Cu"))
+  (gr_rect (start 203.91625 105.325) (end 204.91625 106.325)
+    (stroke (width 0) (type solid)) (fill solid) (layer "F.Cu"))
+  (gr_poly
+    (pts
+      (xy 201.91625 106.325)
+      (xy 201.91625 107.325)
+      (xy 199.91625 107.325)
+      (xy 199.91625 108.325)
+      (xy 201.91625 108.325)
+      (xy 201.91625 109.325)
+      (xy 199.91625 109.325)
+      (xy 199.91625 110.325)
+      (xy 201.91625 110.325)
+      (xy 201.91625 109.325)
+      (xy 202.91625 109.325)
+      (xy 202.91625 110.325)
+      (xy 204.91625 110.325)
+      (xy 204.91625 109.325)
+      (xy 202.91625 109.325)
+      (xy 202.91625 108.325)
+      (xy 204.91625 108.325)
+      (xy 204.91625 107.325)
+      (xy 202.91625 107.325)
+      (xy 202.91625 106.325)
+    )
+    (stroke (width 0) (type solid)) (fill solid) (layer "F.Mask"))
+  (gr_rect (start 203.91625 105.325) (end 204.91625 106.325)
+    (stroke (width 0) (type solid)) (fill solid) (layer "F.Mask"))
+  (gr_rect (start 199.91625 105.325) (end 200.91625 106.325)
+    (stroke (width 0) (type solid)) (fill solid) (layer "F.Mask"))
   (gr_line locked (start 313.325 84) (end 310.15 84)
     (stroke (width 0.1) (type default)) (layer "Edge.Cuts"))
@@
   (gr_rect locked (start 28.575 66.675) (end 71.4375 85.725)
     (stroke (width 0.1) (type default)) (fill none) (layer "F.Fab"))
+  (gr_line (start 202.41625 117.15) (end 202.41625 107.825)
+    (stroke (width 0.15) (type default)) (layer "F.Fab"))
   (gr_rect (start 123.925 104.775) (end 242.9875 123.825)
     (stroke (width 0.1) (type default)) (fill none) (layer "F.Fab"))
-  (gr_rect (start 154.78125 104.775) (end 173.83125 123.825)
+  (gr_line (start 211.74125 107.825) (end 202.41625 107.825)
+    (stroke (width 0.15) (type default)) (layer "F.Fab"))
+  (gr_rect locked (start 154.78125 104.775) (end 173.83125 123.825)
     (stroke (width 0.1) (type default)) (fill none) (layer "F.Fab"))
+  (gr_line (start 193.09125 107.825) (end 202.41625 107.825)
+    (stroke (width 0.15) (type default)) (layer "F.Fab"))
   (gr_rect locked (start 28.575 47.625) (end 57.15 66.675)
     (stroke (width 0.1) (type default)) (fill none) (layer "F.Fab"))
   (gr_rect locked (start 290.5125 104.775) (end 314.325 123.825)
     (stroke (width 0.1) (type default)) (fill none) (layer "F.Fab"))
+  (gr_line (start 202.41625 98.5) (end 202.41625 107.825)
+    (stroke (width 0.15) (type default)) (layer "F.Fab"))
   (gr_rect locked (start 242.8875 104.775) (end 266.7 123.825)
     (stroke (width 0.1) (type default)) (fill none) (layer "F.Fab"))
@@
   (gr_rect locked (start 266.7 104.775) (end 290.5125 123.825)
     (stroke (width 0.1) (type default)) (fill none) (layer "F.Fab"))
+  (gr_text locked "0.4.1+20230811" (at 205.91625 107.825) (layer "F.SilkS")
+    (effects (font (size 1 1) (thickness 0.15)) (justify left))
+  )
+  (gr_text locked "JLCJLCJLCJLC" (at 205.91625 109.825) (layer "F.SilkS")
+    (effects (font (size 1 1) (thickness 0.15)) (justify left))
+  )
+  (gr_text locked "Five Octave Keys" (at 205.91625 105.825) (layer "F.SilkS")
+    (effects (font (size 1 1) (thickness 0.15)) (justify left))
+  )
   (dimension locked (type aligned) (layer "Cmts.User")
     (pts (xy 314.325 28.575) (xy 314.325 123.825))
@@
     )
   )
+  (group "" (id 3ed7a372-07f8-4df1-b76a-9618e7c0f1fc)
+    (members
+      67d0b846-1c73-40bf-9b30-a443a45031ca
+      7737486c-865a-4286-a532-99882b1509ae
+      9b7db061-abd3-4bbc-96c3-f3f52a5dd34d
+      ac0c1f77-22b6-4867-ac8e-29193ec4af94
+    )
+  )

Commit message: Fix footprint orientation for PCBA
Parts:
- moved SW31 3.86 mm to (272.1, 72.4), turned to 180 degrees
- moved SW10 3.86 mm to (134.0, 34.3), turned to 180 degrees
- moved SW32 3.86 mm to (253.0, 72.4), turned to 180 degrees
- moved SW35 3.86 mm to (195.9, 72.4), turned to 180 degrees
- moved SW37 3.86 mm to (157.8, 72.4), turned to 180 degrees
- moved SW45 3.86 mm to (243.5, 91.4), turned to 180 degrees
- moved SW47 3.86 mm to (205.4, 91.4), turned to 180 degrees
- moved SW5 3.86 mm to (229.2, 34.3), turned to 180 degrees
- moved SW50 3.86 mm to (148.3, 91.4), turned to 180 degrees
- moved SW58 3.86 mm to (255.4, 110.5), turned to 180 degrees
- moved SW59 3.86 mm to (184.0, 110.5), turned to 180 degrees
- moved SW8 3.86 mm to (172.1, 34.3), turned to 180 degrees
- moved SW11 3.86 mm to (114.9, 34.3), turned to 180 degrees
- moved SW12 3.86 mm to (95.9, 34.3), turned to 180 degrees
- moved SW39 3.86 mm to (119.7, 72.4), turned to 180 degrees
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