File: electronics/Five_Octave_Keys/Five_Octave_Keys.kicad_pcb (KiCad board)
At the start: 2 copper layers, 285.8 x 95.2 mm, 131 parts, among them J1 FFC Connector, SW1 Key Esc, SW10 Key 9, SW11 Key 0, SW12 Key -, SW13 Key =, SW14 Key \, SW15 Key `, SW16 locked, SW17 Key Q, SW18 locked, SW19 Key E, SW2 Key 1, SW20 Key R, SW21 Key T, SW22 Key Y, SW23 Key U, SW24 Key I, SW25 Key O, SW26 Key P, SW27 Key [, SW28 Key ], SW29 Key BS, SW3 Key 2, SW30 Key Caps, SW31 Key A, SW32 Key S, SW33 Key D, SW34 Key F, SW35 Key G, SW36 Key H, SW37 Key J, SW38 Key K, SW39 Key L, SW4 Key 3, SW40 Key ;, SW41 Key ', SW42 Key Return, SW43 Key Shift, SW44 Key Z, SW45 Key X, SW46 Key C, SW47 Key V, SW48 Key B, SW49 Key N, SW5 Key 4, SW50 Key M, SW51 Key ,, SW52 Key ., SW53 Key /, SW54 Key Shift, SW55 Key Fn, SW56 Key Ctrl, SW57 Key Opt, SW58 Key Cmd, SW59 Key Space, SW6 Key 5, SW60 Key Cmd, SW61 Key MO(1), SW7 Key 6, SW8 Key 7, SW9 Key 8

Commit message: Change M2 footprint
Parts:
- removed the REF** at (311.3, 47.6)
- removed the REF** at (311.3, 120.8)
- removed the REF** at (88.7, 120.8)
- removed the REF** at (31.6, 47.6)
- removed the REF** at (31.6, 101.8)
Other:
- outline, holes or cut-outs redrawn
Changed lines of the file:
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@@
     (title "Five Octave - Keys")
     (date "2023-08-14")
-    (rev "1.0.0-wip.1")
+    (rev "1.0.0-wip.2")
     (comment 1 "https://github.com/takayoshiotake/five-octave-61-key-keyboard")
   )
@@
     )
   )
-  (footprint "MountingHole:MountingHole_2.2mm_M2_Pad" (layer "F.Cu")
-    (at 311.325 47.625 180)
-    (descr "Mounting Hole 2.2mm, M2")
-    (tags "mounting hole 2.2mm m2")
-    (attr exclude_from_pos_files exclude_from_bom)
-    (fp_text reference "REF**" (at 0 -3.2) (layer "F.SilkS") hide
-        (effects (font (size 1 1) (thickness 0.15)))
-    )
-    (fp_text value "MountingHole_2.2mm_M2_Pad" (at 0 3.2) (layer "F.Fab") hide
-        (effects (font (size 1 1) (thickness 0.15)))
-    )
-    (fp_text user "${REFERENCE}" (at 0 0) (layer "F.Fab") hide
-        (effects (font (size 1 1) (thickness 0.15)))
-    )
-    (fp_circle (center 0 0) (end 2.2 0)
-      (stroke (width 0.15) (type solid)) (fill none) (layer "Cmts.User"))
-    (fp_circle (center 0 0) (end 2.45 0)
-      (stroke (width 0.05) (type solid)) (fill none) (layer "F.CrtYd"))
-    (pad "1" thru_hole circle (at 0 0 180) (size 4.4 4.4) (drill 2.2) (layers "*.Cu" "*.Mask"))
-  )
   (footprint "Project_Library:D_SOD-323F" locked (layer "F.Cu")
     (at 206.4225 38.1 90)
@@
     )
   )
-  (footprint "MountingHole:MountingHole_2.2mm_M2_Pad" (layer "F.Cu")
-    (at 311.325 120.825 180)
-    (descr "Mounting Hole 2.2mm, M2")
-    (tags "mounting hole 2.2mm m2")
-    (attr exclude_from_pos_files exclude_from_bom)
-    (fp_text reference "REF**" (at 0 -3.2) (layer "F.SilkS") hide
-        (effects (font (size 1 1) (thickness 0.15)))
-    )
-    (fp_text value "MountingHole_2.2mm_M2_Pad" (at 0 3.2) (layer "F.Fab") hide
-        (effects (font (size 1 1) (thickness 0.15)))
-    )
-    (fp_text user "${REFERENCE}" (at 0 0) (layer "F.Fab") hide
-        (effects (font (size 1 1) (thickness 0.15)))
-    )
-    (fp_circle (center 0 0) (end 2.2 0)
-      (stroke (width 0.15) (type solid)) (fill none) (layer "Cmts.User"))
-    (fp_circle (center 0 0) (end 2.45 0)
-      (stroke (width 0.05) (type solid)) (fill none) (layer "F.CrtYd"))
-    (pad "1" thru_hole circle (at 0 0 180) (size 4.4 4.4) (drill 2.2) (layers "*.Cu" "*.Mask"))
-  )
   (footprint "Project_Library:D_SOD-323F" locked (layer "F.Cu")
     (at 87.36 95.25 90)
@@
     )
   )
-  (footprint "MountingHole:MountingHole_2.2mm_M2_Pad" (layer "F.Cu")
-    (at 88.725 120.825 180)
-    (descr "Mounting Hole 2.2mm, M2")
-    (tags "mounting hole 2.2mm m2")
-    (attr exclude_from_pos_files exclude_from_bom)
-    (fp_text reference "REF**" (at 0 -3.2) (layer "F.SilkS") hide
-        (effects (font (size 1 1) (thickness 0.15)))
-    )
-    (fp_text value "MountingHole_2.2mm_M2_Pad" (at 0 3.2) (layer "F.Fab") hide
-        (effects (font (size 1 1) (thickness 0.15)))
-    )
-    (fp_text user "${REFERENCE}" (at 0 0) (layer "F.Fab") hide
-        (effects (font (size 1 1) (thickness 0.15)))
-    )
-    (fp_circle (center 0 0) (end 2.2 0)
-      (stroke (width 0.15) (type solid)) (fill none) (layer "Cmts.User"))
-    (fp_circle (center 0 0) (end 2.45 0)
-      (stroke (width 0.05) (type solid)) (fill none) (layer "F.CrtYd"))
-    (pad "1" thru_hole circle (at 0 0 180) (size 4.4 4.4) (drill 2.2) (layers "*.Cu" "*.Mask"))
-  )
   (footprint "Project_Library:Hot_Swap_Socket_CPG151101S11" locked (layer "F.Cu")
     (at 110.1725 91.44 180)
@@
     )
   )
-  (footprint "MountingHole:MountingHole_2.2mm_M2_Pad" (layer "F.Cu")
-    (at 31.575 47.625 180)
-    (descr "Mounting Hole 2.2mm, M2")
-    (tags "mounting hole 2.2mm m2")
-    (attr exclude_from_pos_files exclude_from_bom)
-    (fp_text reference "REF**" (at 0 -3.2) (layer "F.SilkS") hide
-        (effects (font (size 1 1) (thickness 0.15)))
-    )
-    (fp_text value "MountingHole_2.2mm_M2_Pad" (at 0 3.2) (layer "F.Fab") hide
-        (effects (font (size 1 1) (thickness 0.15)))
-    )
-    (fp_text user "${REFERENCE}" (at 0 0) (layer "F.Fab") hide
-        (effects (font (size 1 1) (thickness 0.15)))
-    )
-    (fp_circle (center 0 0) (end 2.2 0)
-      (stroke (width 0.15) (type solid)) (fill none) (layer "Cmts.User"))
-    (fp_circle (center 0 0) (end 2.45 0)
-      (stroke (width 0.05) (type solid)) (fill none) (layer "F.CrtYd"))
-    (pad "1" thru_hole circle (at 0 0 180) (size 4.4 4.4) (drill 2.2) (layers "*.Cu" "*.Mask"))
-  )
   (footprint "Project_Library:D_SOD-323F" locked (layer "F.Cu")
     (at 46.87875 76.2 90)
@@
     )
   )
-  (footprint "MountingHole:MountingHole_2.2mm_M2_Pad" (layer "F.Cu")
-    (at 31.575 101.775 180)
-    (descr "Mounting Hole 2.2mm, M2")
-    (tags "mounting hole 2.2mm m2")
-    (attr exclude_from_pos_files exclude_from_bom)
-    (fp_text reference "REF**" (at 0 -3.2) (layer "F.SilkS") hide
-        (effects (font (size 1 1) (thickness 0.15)))
-    )
-    (fp_text value "MountingHole_2.2mm_M2_Pad" (at 0 3.2) (layer "F.Fab") hide
-        (effects (font (size 1 1) (thickness 0.15)))
-    )
-    (fp_text user "${REFERENCE}" (at 0 0) (layer "F.Fab") hide
-        (effects (font (size 1 1) (thickness 0.15)))
-    )
-    (fp_circle (center 0 0) (end 2.2 0)
-      (stroke (width 0.15) (type solid)) (fill none) (layer "Cmts.User"))
-    (fp_circle (center 0 0) (end 2.45 0)
-      (stroke (width 0.05) (type solid)) (fill none) (layer "F.CrtYd"))
-    (pad "1" thru_hole circle (at 0 0 180) (size 4.4 4.4) (drill 2.2) (layers "*.Cu" "*.Mask"))
-  )
   (footprint "Project_Library:Hot_Swap_Socket_CPG151101S11" locked (layer "F.Cu")
     (at 167.3225 91.44 180)
@@
   (gr_rect (start 199.91625 105.325) (end 200.91625 106.325)
     (stroke (width 0) (type solid)) (fill solid) (layer "F.Mask"))
+  (gr_circle (center 311.325 120.825) (end 313.075 120.825)
+    (stroke (width 0.1) (type default)) (fill none) (layer "Cmts.User"))
+  (gr_circle (center 311.325 47.625) (end 313.075 47.625)
+    (stroke (width 0.1) (type default)) (fill none) (layer "Cmts.User"))
+  (gr_circle (center 31.575 47.625) (end 33.325 47.625)
+    (stroke (width 0.1) (type default)) (fill none) (layer "Cmts.User"))
+  (gr_circle (center 88.725 120.825) (end 90.475 120.825)
+    (stroke (width 0.1) (type default)) (fill none) (layer "Cmts.User"))
+  (gr_circle (center 31.575 101.775) (end 33.325 101.775)
+    (stroke (width 0.1) (type default)) (fill none) (layer "Cmts.User"))
   (gr_line locked (start 314.325 31.575) (end 314.325 120.825)
     (stroke (width 0.1) (type default)) (layer "Edge.Cuts"))
@@
   (gr_arc locked (start 314.325 120.825) (mid 313.44632 122.94632) (end 311.325 123.825)
     (stroke (width 0.1) (type default)) (layer "Edge.Cuts"))
+  (gr_circle (center 31.575 101.775) (end 32.675 101.775)
+    (stroke (width 0.1) (type default)) (fill none) (layer "Edge.Cuts"))
+  (gr_circle (center 311.325 120.825) (end 312.425 120.825)
+    (stroke (width 0.1) (type default)) (fill none) (layer "Edge.Cuts"))
   (gr_arc locked (start 28.575 31.575) (mid 29.45368 29.45368) (end 31.575 28.575)
     (stroke (width 0.1) (type default)) (layer "Edge.Cuts"))
@@
   (gr_arc locked (start 84.725 104.775) (mid 85.432107 105.067893) (end 85.725 105.775)
     (stroke (width 0.1) (type default)) (layer "Edge.Cuts"))
+  (gr_circle (center 31.575 47.625) (end 32.675 47.625)
+    (stroke (width 0.1) (type default)) (fill none) (layer "Edge.Cuts"))
+  (gr_circle (center 311.325 47.625) (end 312.425 47.625)
+    (stroke (width 0.1) (type default)) (fill none) (layer "Edge.Cuts"))
+  (gr_circle (center 88.725 120.825) (end 89.825 120.825)
+    (stroke (width 0.1) (type default)) (fill none) (layer "Edge.Cuts"))
   (gr_line locked (start 28.575 101.775) (end 28.575 31.575)
     (stroke (width 0.1) (type default)) (layer "Edge.Cuts"))
+  (gr_circle (center 88.725 120.825) (end 90.725 120.825)
+    (stroke (width 0.1) (type default)) (fill none) (layer "F.CrtYd"))
+  (gr_circle (center 311.325 47.625) (end 313.325 47.625)
+    (stroke (width 0.1) (type default)) (fill none) (layer "F.CrtYd"))
+  (gr_circle (center 311.325 120.825) (end 313.325 120.825)
+    (stroke (width 0.1) (type default)) (fill none) (layer "F.CrtYd"))
+  (gr_circle (center 31.575 47.625) (end 33.575 47.625)
+    (stroke (width 0.1) (type default)) (fill none) (layer "F.CrtYd"))
+  (gr_circle (center 31.575 101.775) (end 33.575 101.775)
+    (stroke (width 0.1) (type default)) (fill none) (layer "F.CrtYd"))
   (gr_rect locked (start 285.75 47.625) (end 314.325 66.675)
     (stroke (width 0.1) (type default)) (fill none) (layer "F.Fab"))
@@
   (gr_rect locked (start 266.7 104.775) (end 290.5125 123.825)
     (stroke (width 0.1) (type default)) (fill none) (layer "F.Fab"))
-  (gr_text locked "0.4.1+20230812" (at 205.91625 107.825) (layer "F.SilkS")
+  (gr_text locked "1.0.0+20230814" (at 205.91625 107.825) (layer "F.SilkS")
     (effects (font (size 1 1) (thickness 0.15)) (justify left))
   )
@@
     )
   )
+  (group "" (id 518df08a-1c37-463f-ac76-18ababff3e0a)
+    (members
+      4042e5c5-3693-40d6-bf01-9217dacd43f9
+      667578cc-a68c-4e2d-a9d3-859dbbf830a5
+      c5c138ad-651e-4a44-8950-0a46cb25d358
+    )
+  )
+  (group "" (id 71db6ef8-655f-4a2f-83ef-f92c0a5da85b)
+    (members
+      3bd20103-89d8-4243-90fc-3deaa12a6070
+      5c831af0-6efc-4ec3-88d3-2d2dc47aa10f
+      a5b49e3d-10bd-436d-be18-5dff0bb8e31b
+    )
+  )
+  (group "" (id af87dcec-ebee-44ea-b655-7cdbd72b37c8)
+    (members
+      66e61838-3d48-490d-825b-3d19ceae3fe7
+      83fa86c3-59a1-4950-afff-fcc8cb0fa011
+      c1c0f7ff-489d-44d2-9a54-ab10252b46d8
+    )
+  )
+  (group "" (id b558eb1c-8dc8-4f92-8777-5a437517edb4)
+    (members
+      956bd340-d557-43ac-9a3e-5e6564eabc37
+      b1d03439-d07a-495e-9629-d57f1d51db04
+      f5b9c718-40b6-4cb9-8a15-ed983739009b
+    )
+  )
+  (group "" (id b6ed2d45-e45b-44ee-9f23-b6cb4a4c7efb)
+    (members
+      24186877-bdb4-4b94-a5e3-166d513be1c0
+      6cfd8575-9866-464d-9e48-b0c45c5f3f6c
+      e7fd8863-3e31-468d-aa2d-6dce9850018c
+    )
+  )

Commit message: Fix Shift and Fn key size
Parts:
- moved SW54 7.14 mm to (64.9, 91.4)
- moved D54 7.14 mm to (61.2, 95.2)
- moved D55 7.14 mm to (35.0, 95.2)
- moved SW55 7.14 mm to (38.7, 91.4)
Routing:
- net COL5: track 360.7 -> 375.0 mm
- net ROW7: track 176.8 -> 183.9 mm
- net COL6: track 369.8 -> 365.9 mm
- net ROW6: track 216.6 -> 218.6 mm, vias 2 -> 4
- net COL7: track 353.8 -> 354.6 mm
Other:
- outline, holes or cut-outs redrawn

Commit message: Modify outline curve
Other:
- outline, holes or cut-outs redrawn
Changed lines of the file:
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@@
     (title "Five Octave - Keys")
     (date "2023-08-15")
-    (rev "1.0.0-wip.3")
+    (rev "1.0.0-wip.4")
     (comment 1 "https://github.com/takayoshiotake/five-octave-61-key-keyboard")
   )
@@
   (gr_circle (center 51.196875 101.775) (end 52.946875 101.775)
     (stroke (width 0.1) (type default)) (fill none) (layer "Cmts.User"))
-  (gr_line locked (start 314.325 31.575) (end 314.325 120.825)
+  (gr_arc (start 86.725 123.825) (mid 86.017893 123.532107) (end 85.725 122.825)
     (stroke (width 0.1) (type default)) (layer "Edge.Cuts"))
-  (gr_arc locked (start 88.725 123.825) (mid 86.60368 122.94632) (end 85.725 120.825)
+  (gr_arc locked (start 28.575 29.575) (mid 28.867893 28.867893) (end 29.575 28.575)
     (stroke (width 0.1) (type default)) (layer "Edge.Cuts"))
-  (gr_line locked (start 85.725 105.775) (end 85.725 120.825)
+  (gr_line (start 314.325 29.575) (end 314.325 122.825)
     (stroke (width 0.1) (type default)) (layer "Edge.Cuts"))
-  (gr_arc locked (start 31.575 104.775) (mid 29.45368 103.89632) (end 28.575 101.775)
+  (gr_arc (start 313.325 28.575) (mid 314.032107 28.867893) (end 314.325 29.575)
     (stroke (width 0.1) (type default)) (layer "Edge.Cuts"))
-  (gr_arc locked (start 311.325 28.575) (mid 313.44632 29.45368) (end 314.325 31.575)
+  (gr_line (start 85.725 105.775) (end 85.725 122.825)
     (stroke (width 0.1) (type default)) (layer "Edge.Cuts"))
-  (gr_line locked (start 311.325 123.825) (end 88.725 123.825)
-    (stroke (width 0.1) (type default)) (layer "Edge.Cuts"))
-  (gr_arc locked (start 314.325 120.825) (mid 313.44632 122.94632) (end 311.325 123.825)
+  (gr_line (start 313.325 123.825) (end 86.725 123.825)
     (stroke (width 0.1) (type default)) (layer "Edge.Cuts"))
   (gr_circle (center 51.196875 101.775) (end 52.296875 101.775)
@@
   (gr_circle (center 290.5125 120.825) (end 291.6125 120.825)
     (stroke (width 0.1) (type default)) (fill none) (layer "Edge.Cuts"))
-  (gr_arc locked (start 28.575 31.575) (mid 29.45368 29.45368) (end 31.575 28.575)
+  (gr_line (start 84.725 104.775) (end 29.575 104.775)
     (stroke (width 0.1) (type default)) (layer "Edge.Cuts"))
-  (gr_line locked (start 84.725 104.775) (end 31.575 104.775)
+  (gr_arc (start 29.575 104.775) (mid 28.867893 104.482107) (end 28.575 103.775)
     (stroke (width 0.1) (type default)) (layer "Edge.Cuts"))
-  (gr_line locked (start 31.575 28.575) (end 311.325 28.575)
+  (gr_line locked (start 29.575 28.575) (end 313.325 28.575)
     (stroke (width 0.1) (type default)) (layer "Edge.Cuts"))
   (gr_arc locked (start 84.725 104.775) (mid 85.432107 105.067893) (end 85.725 105.775)
@@
   (gr_circle (center 311.325 47.625) (end 312.425 47.625)
     (stroke (width 0.1) (type default)) (fill none) (layer "Edge.Cuts"))
+  (gr_arc (start 314.325 122.825) (mid 314.032107 123.532107) (end 313.325 123.825)
+    (stroke (width 0.1) (type default)) (layer "Edge.Cuts"))
   (gr_circle (center 142.875 120.825) (end 143.975 120.825)
     (stroke (width 0.1) (type default)) (fill none) (layer "Edge.Cuts"))
-  (gr_line locked (start 28.575 101.775) (end 28.575 31.575)
+  (gr_line (start 28.575 103.775) (end 28.575 29.575)
     (stroke (width 0.1) (type default)) (layer "Edge.Cuts"))
   (gr_circle (center 142.875 120.825) (end 144.875 120.825)
@@
     )
   )
-  (group "" locked (id 2b7a5d49-ce1f-4f4f-a451-986d00f426c2)
-    (members
-      17e6a2cc-fa3a-4bb1-be4b-56d10572eeba
-      3411936c-3f5b-4264-925a-acdbc19e1790
-      6b89fc0b-0054-4fe1-b1ac-e86981c65b0e
-      aaa7eeb2-4c00-43f2-8d5d-69ebd72b8237
-      b380686c-5b2b-4969-b28b-fdedab3ee9e9
-      f0216085-a6bc-4e96-8b5f-8405d197d0de
-    )
-  )
