File: electronics/Five_Octave_MCU/Five_Octave_MCU.kicad_pcb (KiCad board)
At the start: 2 copper layers, 0 parts

Commit message: WIP
Parts:
- added C1: 30pF, Capacitor_SMD:C_0402_1005Metric, F.Cu at (32.5, 51.8)
- added C10: 0.1uF, Capacitor_SMD:C_0402_1005Metric, F.Cu at (44.1, 38.8)
- added C11: 0.1uF, Capacitor_SMD:C_0402_1005Metric, F.Cu at (39.2, 35.6)
- added C12: 0.1uF, Capacitor_SMD:C_0402_1005Metric, F.Cu at (38.2, 35.6)
- added C13: 0.1uF, Capacitor_SMD:C_0402_1005Metric, F.Cu at (39.4, 48.8)
- added C14: 0.1uF, Capacitor_SMD:C_0402_1005Metric, F.Cu at (37.2, 35.6)
- added C15: 10uF, Capacitor_SMD:C_0402_1005Metric, F.Cu at (33.5, 28.7)
- added C16: 10uF, Capacitor_SMD:C_0402_1005Metric, F.Cu at (34.5, 33.7)
- added C2: 30pF, Capacitor_SMD:C_0402_1005Metric, F.Cu at (32.5, 53.8)
- added C3: 1uF, Capacitor_SMD:C_0402_1005Metric, F.Cu at (43.2, 36.5)
- added C4: 1uF, Capacitor_SMD:C_0402_1005Metric, F.Cu at (42.2, 36.5)
- added C5: 0.1uF, Capacitor_SMD:C_0402_1005Metric, F.Cu at (34.0, 39.8)
- added C6: 0.1uF, Capacitor_SMD:C_0402_1005Metric, F.Cu at (33.2, 43.8)
- added C7: 0.1uF, Capacitor_SMD:C_0402_1005Metric, F.Cu at (38.4, 48.8)
- added C8: 0.1uF, Capacitor_SMD:C_0402_1005Metric, F.Cu at (44.7, 43.8)
- added C9: 0.1uF, Capacitor_SMD:C_0402_1005Metric, F.Cu at (44.1, 39.8)
- added J1: HRO_TYPE-C-31-M-12, Project_Library:HRO_TYPE-C-31-M-12, F.Cu at (40.0, 30.0)
- added J2: FFC Connector, Project_Library:JUSHUO_AFC01-S16FCC-00, F.Cu at (49.8, 43.8)
- added LED1: WS2812C-2020-V1, Project_Library:WS2812C-2020, F.Cu at (28.0, 48.8)
- added R1: 10K, Resistor_SMD:R_0402_1005Metric, F.Cu at (41.5, 47.4)
- added R2: 1K, Resistor_SMD:R_0402_1005Metric, F.Cu at (38.3, 52.6)
- added R3: 10K, Resistor_SMD:R_0402_1005Metric, F.Cu at (30.7, 33.7)
- added R4: 1K, Resistor_SMD:R_0402_1005Metric, F.Cu at (29.1, 40.7)
- added R5: 27, Resistor_SMD:R_0402_1005Metric, F.Cu at (40.2, 36.5)
- added R6: 27, Resistor_SMD:R_0402_1005Metric, F.Cu at (41.2, 36.5)
- added R7: 5.1K, Resistor_SMD:R_0402_1005Metric, F.Cu at (38.0, 34.1)
- added R8: 5.1K, Resistor_SMD:R_0402_1005Metric, F.Cu at (42.0, 34.1)
- added SW1: Alps_Alpine_SKRP, Project_Library:Tactile_Switch_SKRP_Series, F.Cu at (44.0, 52.5)
- added SW2: Alps_Alpine_SKRP, Project_Library:Tactile_Switch_SKRP_Series, F.Cu at (28.0, 44.5)
- added U1: Raspberry_Pi_RP2040, Project_Library:RP2040_QFN-56, F.Cu at (39.0, 42.6)
- added U2: W25Q64JVXGIQ, Project_Library:XSON-8-EP_4x4mm, F.Cu at (32.1, 36.4)
- added U3: AP2112K-3.3, Package_TO_SOT_SMD:SOT-23-5, F.Cu at (33.0, 31.2)
- added Y1: 12MHz, Crystal:Crystal_SMD_3225-4Pin_3.2x2.5mm, F.Cu at (35.8, 52.6)
Routing:
- net +3V3: track 0.00 -> 70.1 mm, vias 0 -> 5
- net GND: track 0.00 -> 20.4 mm, vias 0 -> 18
- net +1V1: track 0.00 -> 18.8 mm, vias 0 -> 2
- net +5V: track 0.00 -> 17.2 mm
- net QSPI_SS_N: track 0.00 -> 16.2 mm
- net Net-(U1-QSPI_SD1): track 0.00 -> 13.0 mm
- net Net-(U1-QSPI_SD2): track 0.00 -> 12.1 mm
- net ROW2: track 0.00 -> 8.14 mm
- net ROW3: track 0.00 -> 7.07 mm
- net Net-(U1-QSPI_SD3): track 0.00 -> 6.51 mm
- net Net-(J1-D--PadA7): track 0.00 -> 6.51 mm
- net ROW7: track 0.00 -> 6.37 mm
- net ROW6: track 0.00 -> 6.33 mm
- net ROW5: track 0.00 -> 6.29 mm
- net COL7: track 0.00 -> 6.21 mm
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- added copper zone on F.Cu, net +3V3
- added copper zone on B.Cu, net GND
- added copper zone on F.Cu, net GND
Other:
- board outline added: 28.6 x 28.6 mm
- board text added: "B"
- board text added: "R"
