File: electronics/Five_Octave_MCU/Five_Octave_MCU.kicad_pcb (KiCad board)
At the start: 2 copper layers, 28.6 x 28.6 mm, 33 parts, among them J1 HRO_TYPE-C-31-M-12, J2 FFC Connector, SW1 Alps_Alpine_SKRP, SW2 Alps_Alpine_SKRP, U1 Raspberry_Pi_RP2040, U2 W25Q64JVXGIQ, U3 AP2112K-3.3, Y1 12MHz

Commit message: WIP
Parts:
- moved C2 2.79 mm to (32.5, 51.0), turned to 180 degrees
- moved C1 2.57 mm to (32.5, 49.3), turned to 180 degrees
- moved Y1 2.49 mm to (35.7, 50.1)
- moved R2 1.22 mm to (37.1, 52.5), turned to 180 degrees
- moved C13 0.45 mm to (39.6, 49.2)
- moved C7 0.45 mm to (38.6, 49.2)
Connections:
- U1 pad 17: unconnected-(U1-GPIO14-Pad17) -> ROW0
- U1 pad 18: unconnected-(U1-GPIO15-Pad18) -> ROW1
Routing:
- net ROW0: track 0.75 -> 15.4 mm, vias 0 -> 2
- net ROW1: track 0.75 -> 14.7 mm, vias 0 -> 2
- net Net-(U1-XIN): track 0.00 -> 8.33 mm
- net Net-(U1-XOUT): track 0.00 -> 6.79 mm
- net NEOPIX_POWER: track 1.46 -> 8.06 mm
- net NEOPIX: track 2.26 -> 8.58 mm
- net Net-(C2-Pad1): track 0.00 -> 4.12 mm
- net GND: track 20.4 -> 23.7 mm, vias 18 -> 21
- net +3V3: track 70.1 -> 73.1 mm
- net +1V1: track 18.8 -> 21.5 mm
- net unconnected-(U1-GPIO10-Pad13): track 2.08 -> 0.00 mm
- net unconnected-(U1-GPIO9-Pad12): track 2.08 -> 0.00 mm
- net unconnected-(U1-GPIO8-Pad11): track 2.08 -> 0.00 mm
Other:
- board text added: "+20230814"
- board text added: "0.1.0"
- board text added: "Five Octave MCU"
- board text added: "JLCJLCJLCJLC"
