File: electronics/Five_Octave_MCU/Five_Octave_MCU.kicad_pcb (KiCad board)
At the start: 2 copper layers, 28.6 x 28.6 mm, 33 parts, among them J1 HRO_TYPE-C-31-M-12, J2 FFC Connector, SW1 Alps_Alpine_SKRP, SW2 Alps_Alpine_SKRP, U1 Raspberry_Pi_RP2040, U2 W25Q64JVXGIQ, U3 AP2112K-3.3, Y1 12MHz

Commit message: Update Five_Octave_MCU.kicad_pcb
Other:
- board text added: "1.0.0"
- board text removed: "0.1.0"
Changed lines of the file:
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@@
     (title "Five Octave - MCU")
     (date "2023-08-14")
-    (rev "1.0.0-wip.3")
+    (rev "1.0.0-wip.4")
     (comment 1 "https://github.com/takayoshiotake/five-octave-61-key-keyboard")
   )
@@
   (gr_line (start 40.43 46.0375) (end 40.43 47.815)
     (stroke (width 0.2) (type default)) (layer "F.Fab"))
-  (gr_text "0.1.0" (at 26.1095 38.896643 90) (layer "F.SilkS")
+  (gr_text "1.0.0" (at 26.1095 38.896643 90) (layer "F.SilkS")
     (effects (font (size 1 1) (thickness 0.15)) (justify left top))
   )
