File: electronics/Five_Octave_MCU/Five_Octave_MCU.kicad_pcb (KiCad board)
At the start: 2 copper layers, 28.6 x 28.6 mm, 33 parts, among them J1 HRO_TYPE-C-31-M-12, J2 FFC Connector, SW1 Alps_Alpine_SKRP, SW2 Alps_Alpine_SKRP, U1 Raspberry_Pi_RP2040, U2 W25Q64JVXGIQ, U3 AP2112K-3.3, Y1 12MHz

Commit message: Fix FFC connector assignment
Connections:
- J2 pad 1: ROW0 -> COL7
- J2 pad 10: COL1 -> ROW6
- J2 pad 11: COL2 -> ROW5
- J2 pad 12: COL3 -> ROW4
- J2 pad 13: COL4 -> ROW3
- J2 pad 14: COL5 -> ROW2
- J2 pad 15: COL6 -> ROW1
- J2 pad 16: COL7 -> ROW0
- J2 pad 2: ROW1 -> COL6
- J2 pad 3: ROW2 -> COL5
- J2 pad 4: ROW3 -> COL4
- J2 pad 5: ROW4 -> COL3
- J2 pad 6: ROW5 -> COL2
- J2 pad 7: ROW6 -> COL1
- J2 pad 8: ROW7 -> COL0
- J2 pad 9: COL0 -> ROW7
- U1 pad 17: ROW0 -> COL7
- U1 pad 18: ROW1 -> COL6
- U1 pad 27: ROW2 -> COL5
- U1 pad 28: ROW3 -> COL4
- U1 pad 29: ROW4 -> COL3
- U1 pad 30: ROW5 -> COL2
- U1 pad 31: ROW6 -> COL1
- U1 pad 32: ROW7 -> COL0
- U1 pad 34: COL0 -> ROW7
- U1 pad 35: COL1 -> ROW6
- U1 pad 36: COL2 -> ROW5
- U1 pad 37: COL3 -> ROW4
- U1 pad 38: COL4 -> ROW3
- U1 pad 39: COL5 -> ROW2
- U1 pad 40: COL6 -> ROW1
- U1 pad 41: COL7 -> ROW0
Routing:
- net ROW0: track 15.4 -> 6.21 mm, vias 2 -> 0
- net COL7: track 6.21 -> 15.4 mm, vias 0 -> 2
- net ROW1: track 14.7 -> 6.16 mm, vias 2 -> 0
- net COL6: track 6.16 -> 14.7 mm, vias 0 -> 2
- net ROW2: track 8.14 -> 6.12 mm
- net COL5: track 6.12 -> 8.14 mm
- net ROW3: track 7.07 -> 6.08 mm
- net COL4: track 6.08 -> 7.07 mm

Commit message: Change footprint for AP2112K-3.3
Parts:
- U3: footprint Package_TO_SOT_SMD:SOT-23-5 -> Project_Library:SOT-23-5
- turned U3 to 180 degrees
Changed lines of the file:
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@@
   (title_block
     (title "Five Octave - MCU")
-    (date "2023-08-15")
-    (rev "1.0.0-wip.7")
+    (date "2023-08-21")
+    (rev "1.0.0")
     (comment 1 "https://github.com/takayoshiotake/five-octave-61-key-keyboard")
   )
@@
     )
   )
-  (footprint "Package_TO_SOT_SMD:SOT-23-5" (layer "F.Cu")
-    (at 33.0465 31.1825 -90)
+  (footprint "Project_Library:SOT-23-5" (layer "F.Cu")
+    (at 33.0465 31.1825 180)
     (descr "SOT, 5 Pin (https://www.jedec.org/sites/default/files/docs/Mo-178c.PDF variant AA), generated with kicad-footprint-generator ipc_gullwing_generator.py")
     (tags "SOT TO_SOT_SMD")
@@
     (property "ki_keywords" "linear regulator ldo fixed positive")
     (attr smd)
-    (fp_text reference "U3" (at 0 -2.4 90) (layer "F.SilkS") hide
-        (effects (font (size 1 1) (thickness 0.15)))
-    )
-    (fp_text value "AP2112K-3.3" (at 0 2.4 90) (layer "F.Fab") hide
-        (effects (font (size 1 1) (thickness 0.15)))
-    )
-    (fp_text user "${REFERENCE}" (at 0 0 90) (layer "F.Fab")
+    (fp_text reference "U3" (at 0 -2.8) (layer "F.SilkS") hide
+        (effects (font (size 1 1) (thickness 0.15)))
+    )
+    (fp_text value "AP2112K-3.3" (at 0 2.8) (layer "F.Fab") hide
+        (effects (font (size 1 1) (thickness 0.15)))
+    )
+    (fp_text user "${REFERENCE}" (at 0 0) (layer "F.Fab")
         (effects (font (size 0.4 0.4) (thickness 0.06)))
     )
-    (fp_line (start 0 -1.56) (end -1.8 -1.56)
-      (stroke (width 0.12) (type solid)) (layer "F.SilkS"))
-    (fp_line (start 0 -1.56) (end 0.8 -1.56)
-      (stroke (width 0.12) (type solid)) (layer "F.SilkS"))
-    (fp_line (start 0 1.56) (end -0.8 1.56)
-      (stroke (width 0.12) (type solid)) (layer "F.SilkS"))
-    (fp_line (start 0 1.56) (end 0.8 1.56)
-      (stroke (width 0.12) (type solid)) (layer "F.SilkS"))
-    (fp_line (start -2.05 -1.7) (end -2.05 1.7)
-      (stroke (width 0.05) (type solid)) (layer "F.CrtYd"))
-    (fp_line (start -2.05 1.7) (end 2.05 1.7)
-      (stroke (width 0.05) (type solid)) (layer "F.CrtYd"))
-    (fp_line (start 2.05 -1.7) (end -2.05 -1.7)
-      (stroke (width 0.05) (type solid)) (layer "F.CrtYd"))
-    (fp_line (start 2.05 1.7) (end 2.05 -1.7)
-      (stroke (width 0.05) (type solid)) (layer "F.CrtYd"))
-    (fp_line (start -0.8 -1.05) (end -0.4 -1.45)
-      (stroke (width 0.1) (type solid)) (layer "F.Fab"))
-    (fp_line (start -0.8 1.45) (end -0.8 -1.05)
-      (stroke (width 0.1) (type solid)) (layer "F.Fab"))
-    (fp_line (start -0.4 -1.45) (end 0.8 -1.45)
-      (stroke (width 0.1) (type solid)) (layer "F.Fab"))
-    (fp_line (start 0.8 -1.45) (end 0.8 1.45)
-      (stroke (width 0.1) (type solid)) (layer "F.Fab"))
-    (fp_line (start 0.8 1.45) (end -0.8 1.45)
-      (stroke (width 0.1) (type solid)) (layer "F.Fab"))
-    (pad "1" smd roundrect (at -1.1375 -0.95 270) (size 1.325 0.6) (layers "F.Cu" "F.Paste" "F.Mask") (roundrect_rratio 0.25)
+    (fp_line (start -1.56 0) (end -1.56 -0.8)
+      (stroke (width 0.12) (type solid)) (layer "F.SilkS"))
+    (fp_line (start -1.56 0) (end -1.56 1.8)
+      (stroke (width 0.12) (type solid)) (layer "F.SilkS"))
+    (fp_line (start 1.56 0) (end 1.56 -0.8)
+      (stroke (width 0.12) (type solid)) (layer "F.SilkS"))
+    (fp_line (start 1.56 0) (end 1.56 0.8)
+      (stroke (width 0.12) (type solid)) (layer "F.SilkS"))
+    (fp_line (start -1.7 -2.05) (end -1.7 2.05)
+      (stroke (width 0.05) (type solid)) (layer "F.CrtYd"))
+    (fp_line (start -1.7 2.05) (end 1.7 2.05)
+      (stroke (width 0.05) (type solid)) (layer "F.CrtYd"))
+    (fp_line (start 1.7 -2.05) (end -1.7 -2.05)
+      (stroke (width 0.05) (type solid)) (layer "F.CrtYd"))
+    (fp_line (start 1.7 2.05) (end 1.7 -2.05)
+      (stroke (width 0.05) (type solid)) (layer "F.CrtYd"))
+    (fp_line (start -1.45 -0.8) (end 1.45 -0.8)
+      (stroke (width 0.1) (type solid)) (layer "F.Fab"))
+    (fp_line (start -1.45 0.4) (end -1.45 -0.8)
+      (stroke (width 0.1) (type solid)) (layer "F.Fab"))
+    (fp_line (start -1.05 0.8) (end -1.45 0.4)
+      (stroke (width 0.1) (type solid)) (layer "F.Fab"))
+    (fp_line (start 1.45 -0.8) (end 1.45 0.8)
+      (stroke (width 0.1) (type solid)) (layer "F.Fab"))
+    (fp_line (start 1.45 0.8) (end -1.05 0.8)
+      (stroke (width 0.1) (type solid)) (layer "F.Fab"))
+    (pad "1" smd roundrect (at -0.95 1.1375 270) (size 1.325 0.6) (layers "F.Cu" "F.Paste" "F.Mask") (roundrect_rratio 0.25)
       (net 6 "+5V") (pinfunction "VIN") (pintype "power_in"))
-    (pad "2" smd roundrect (at -1.1375 0 270) (size 1.325 0.6) (layers "F.Cu" "F.Paste" "F.Mask") (roundrect_rratio 0.25)
+    (pad "2" smd roundrect (at 0 1.1375 270) (size 1.325 0.6) (layers "F.Cu" "F.Paste" "F.Mask") (roundrect_rratio 0.25)
       (net 2 "GND") (pinfunction "GND") (pintype "power_in"))
-    (pad "3" smd roundrect (at -1.1375 0.95 270) (size 1.325 0.6) (layers "F.Cu" "F.Paste" "F.Mask") (roundrect_rratio 0.25)
+    (pad "3" smd roundrect (at 0.95 1.1375 270) (size 1.325 0.6) (layers "F.Cu" "F.Paste" "F.Mask") (roundrect_rratio 0.25)
       (net 6 "+5V") (pinfunction "EN") (pintype "input"))
-    (pad "4" smd roundrect (at 1.1375 0.95 270) (size 1.325 0.6) (layers "F.Cu" "F.Paste" "F.Mask") (roundrect_rratio 0.25)
+    (pad "4" smd roundrect (at 0.95 -1.1375 270) (size 1.325 0.6) (layers "F.Cu" "F.Paste" "F.Mask") (roundrect_rratio 0.25)
       (net 61 "unconnected-(U3-NC-Pad4)") (pinfunction "NC") (pintype "no_connect"))
-    (pad "5" smd roundrect (at 1.1375 -0.95 270) (size 1.325 0.6) (layers "F.Cu" "F.Paste" "F.Mask") (roundrect_rratio 0.25)
+    (pad "5" smd roundrect (at -0.95 -1.1375 270) (size 1.325 0.6) (layers "F.Cu" "F.Paste" "F.Mask") (roundrect_rratio 0.25)
       (net 4 "+3V3") (pinfunction "VOUT") (pintype "power_out"))
     (model "${KICAD6_3DMODEL_DIR}/Package_TO_SOT_SMD.3dshapes/SOT-23-5.wrl"

Commit message: Update build number
Other:
- board text added: "+20230821"
- board text removed: "+20230814"
Changed lines of the file:
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@@
     (effects (font (size 1 1) (thickness 0.15)) (justify right bottom))
   )
-  (gr_text "+20230814" (at 27.6095 38.896643 90) (layer "F.SilkS")
+  (gr_text "+20230821" (at 27.6095 38.896643 90) (layer "F.SilkS")
     (effects (font (size 1 1) (thickness 0.15)) (justify left top))
   )
