File: mechanics/Five_Octave_Plate/Five_Octave_Plate.kicad_pcb (KiCad board)
At the start: 2 copper layers, 290.8 x 100.3 mm, 0 parts

Commit message: Improve edge-cuts layer
Other:
- outline, holes or cut-outs redrawn

Commit message: Modify outline curve
Other:
- outline, holes or cut-outs redrawn

Commit message: Update version
Other:
- board text added: "1.0.0+20230821"
- board text removed: "1.0.0+20230815"
Changed lines of the file:
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@@
   (title_block
     (title "Five Octave - Plate")
-    (date "2023-08-15")
-    (rev "1.0.0-wip.3")
+    (date "2023-08-21")
+    (rev "1.0.0")
     (comment 1 "https://github.com/takayoshiotake/five-octave-61-key-keyboard")
   )
@@
     )
     (stroke (width 0.1) (type solid)) (fill none) (layer "User.3"))
-  (gr_text "1.0.0+20230815" (at 177.59375 109.8) (layer "F.SilkS")
+  (gr_text "1.0.0+20230821" (at 177.59375 109.8) (layer "F.SilkS")
     (effects (font (size 1 1) (thickness 0.15)) (justify left))
   )
